File: payload.kicad_sch (KiCad schematic)
At the start: 0 parts

Commit message: adds payload wiring diagram mockup
Other:
- note added: "3x Cameras"
- note added: "Antenna"
- note added: "Avionics"
- note added: "Camera Breakout PCB"
- note added: "EPS 1"
- note added: "EPS 2"
- note added: "Magnetic POGO Pin Connector"
- note added: "Payload Bay"
- note added: "RGX Data PCB"
- note added: "RGX Sensors"
- note added: "Recovery Beacon"
- note added: "VTX (Video Transmitter)"
