File: payload.kicad_sch (KiCad schematic)
At the start: 0 parts

Commit message: replaces text with text boxes
Other:
- note removed: "3x Cameras"
- note removed: "Antenna"
- note removed: "Avionics"
- note removed: "Camera Breakout PCB"
- note removed: "EPS 1"
- note removed: "EPS 2"
- note removed: "Magnetic POGO Pin Connector"
- note removed: "Payload Bay"
- note removed: "RGX Data PCB"
- note removed: "RGX Sensors"
- note removed: "Recovery Beacon"
- note removed: "VTX (Video Transmitter)"
