File: payload.kicad_sch (KiCad schematic)
At the start: 0 parts

Commit message: preliminary final
Other:
- note added: "termination"
- note removed: "3x Cameras"
- note removed: "Antenna"
- note removed: "Avionics"
- note removed: "Camera Breakout PCB"
- note removed: "EPS 1"
- note removed: "EPS 2"
- note removed: "Magnetic POGO Pin Connector"
- note removed: "Payload Bay"
- note removed: "RGX Data PCB"
- note removed: "RGX Sensors"
- note removed: "Recovery Beacon"
- note removed: "VTX (Video Transmitter)"

Commit message: payload final?
Other:
- note added: "CHECKLIST [ ] EPS1_J1 - MCP9700 [ ] EPS1_J2 - MCP9700 [ ] EPS1_J3 - CHARGER [ ] EPS1_J4 - ESP32_J2 [ ] EPS1_J6 - TERMINATION [ ] EPS1_J7 - CAM_BREAKOUT_J2 [ ] EPS1_J8 - CAM_BREAKOUT_J1 [ ] EPS1_J1 - MCP9700 [ ] EPS1_J2 - MCP9700 [ ] EPS1_J3 - CHARGER [ ] EPS1_J4 - ESP32_J3 [ ] EPS1_J6 - TERMINATION [ ] EPS1_J7 - CICADA_J1 [ ] EPS1_J8 - ESP32_J1 [ ] CAM_BREAKOUT_J3 - CAM1_J1 [ ] CAM_BREAKOUT_J4 - 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"
- note added: "MCMASTER ROCKETRY"
- note added: "PAYLOAD WIRING DIAGRAM"
- company: (none) -> MCMASTER ROCKETRY
- title: (none) -> PAYLOAD WIRING DIAGRAM
