File: RocketryWiringDiagram.kicad_sch (KiCad schematic)
At the start: 23 parts, among them SW10 SW_DPST_x2, SW11 SW_DPST_x2, SW12 SW_DPST_x2, SW7 SW_DPST_x2, SW8 SW_DPST_x2, SW9 SW_DPST_x2, U1 ADG417BN, U10 ADG417BN, U11 ADG417BN, U12 ADG417BN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

Commit message: clean repo and add payload subsheets
Parts:
- removed BT1, BT2, BT3, BT4, BT5, BT6: Battery_Cell, symbol Device:Battery_Cell
- removed F10, F11, F12, F7, F8, F9: E-Match, symbol Device:Fuse
- removed SW10, SW11, SW12, SW7, SW8, SW9: SW_DPST_x2, symbol Switch:SW_DPST_x2
- removed U1, U10, U11, U12, U2: ADG417BN, Package_DIP:DIP-8_W7.62mm, symbol Analog_Switch:ADG417BN
Other:
- added sheet Controls (controls.kicad_sch)
- added sheet Payload (payload.kicad_sch)
- note removed: "(Relays shown here are actually mosfets, they close the circuit when the control signal is low)"
- note removed: "1S 18650 Battery PCB"
- note removed: "2S 18650 Battery PCB"
- note removed: "4S 18650 Battery PCB"
- note removed: "A In: M1x2 1054301102"
- note removed: "A Out: S1x2"
- note removed: "Air Brake PCB"
- note removed: "Arming Switch PCB"
- note removed: "Arming Switch: S1x2"
- note removed: "B In: M1x2 1054301102"
- note removed: "B Out: S1x2"
- note removed: "Battery: K1x2"
- note removed: "Battery: M1x2 1054301102"
- note removed: "Battery: S1x2"
- note removed: "Blue Raven"
- note removed: "C In: M1x2 1054301102"
- note removed: "C Out: S1x2"
- note removed: "CAN Termination PCB"
- note removed: "Camera PCB"
- note removed: "Drogue: S1x2"
- note removed: "E-Match Adapter Drogue Chute"
- note removed: "E-Match Adapter Main Chute"
- note removed: "E-Match: M2x3 1054051106"
- note removed: "Easy Mini"
- note removed: "Extension: M2x4 1054051108"
- note removed: "Featherweight GPS"
- note removed: "J1x2"
- note removed: "L1x2 534260210"
- note removed: "LR1x2 511630200"
- note removed: "M1x2 1054301102"
- note removed: "MCU STM32"
- note removed: "Main: S1x2"
- note removed: "Payload"
- note removed: "Power Distribution PCB"
- note removed: "R1x2 1053071202"
- note removed: "R1x2 1053072202"
- note removed: "R2x2 1053081204"
- note removed: "R2x3 1053081206"
- note removed: "R2x4 1053051108"
- note removed: "Screw Terminal: S1x6"
- note removed: "Strain Gauges PCB 1"
- note removed: "Strain Gauges PCB 2"
- note removed: "Switches: M2x2 1054051104"
- note removed: "VL Mini"
- note removed: "Void Lake Fusion 4 (Equivalent Electrical Diagram) (Only Circuits Related to E-Matches are Shown)"

Commit message: recovery only wiring diagram
Other:
- added sheet Recovery Only (recovery_only.kicad_sch)
Changed lines of the file:
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@@
 	(paper "A4")
+	(sheet
+		(at 29.21 99.06)
+		(size 36.83 46.99)
+		(fields_autoplaced yes)
+		(stroke
+			(width 0.1524)
+			(type solid)
+		)
+		(fill
+			(color 0 0 0 0.0000)
+		)
+		(property "Sheetname" "Recovery Only"
+			(at 29.21 98.3484 0)
+			(effects
+				(font
+					(size 1.27 1.27)
+				)
+				(justify left bottom)
+			)
+		)
+		(property "Sheetfile" "recovery_only.kicad_sch"
+			(at 29.21 146.6346 0)
+			(effects
+				(font
+					(size 1.27 1.27)
+				)
+				(justify left top)
+			)
+		)
+		(instances
+			(project "RocketryWiringDiagram"
+				(path "/395837be-e671-47e6-8fb9-877478f5d46e"
+					(page "4")
+				)
+			)
+		)
+	)
 	(sheet
 		(at 82.55 36.83)
