File: controls.kicad_sch (KiCad schematic)
At the start: 9 parts

Commit message: controls wiring diagram
Parts:
- removed BT10, BT11, BT12, BT17, BT3, BT4, BT5, BT6, BT8: Battery_Cell, symbol Device:Battery_Cell
- added BT1, BT18, BT2, BT20, BT21, BT22, BT23, BT7, BT9: Battery_Cell, symbol Device:Battery_Cell
Connections:
- new net: BT20.2 (-), BT21.1 (+), BT22.2 (-), BT23.1 (+)
- new net: BT21.2 (-), BT23.2 (-)
- new net: BT20.1 (+), BT22.1 (+)
- new net: BT7.2 (-), BT9.1 (+)
- no-connect marks 1 -> 0
Other:
- note added: "1S 18650"
- note added: "2S 18650"
- note added: "2S2P 18650"
- note added: "Air Brakes"
- note added: "SERVO"
- note removed: "1S 18650 Battery Pack"
- note removed: "2S 18650 Battery Pack"
- note removed: "2S2P 18650 Battery Pack"
- note removed: "VLFX"
