File: controls.kicad_sch (KiCad schematic)
At the start: 9 parts

Commit message: update controls wiring diagram
Connections:
- no-connect marks 0 -> 1
Other:
- note added: "10cm"
- note added: "30cm"
- note added: "5cm"
- note added: "AMP Speed Bridge"
- title: 2024-2025 Avionics Bay Wiring Diagram -> Titan Avionics Bay Wiring Diagram
